File: Main Board/Main Board.sch (KiCad schematic (older format))
At the start: 8 parts, among them J1 Conn_01x04, J2 Conn_02x05_Odd_Even, J3 Conn_01x06, J4 Conn_01x06, J5 Conn_01x02, J6 Conn_01x02

Commit message: Fix BNO055 to use new library
Parts:
- A2: footprint BNO055:BNO055 -> SCR_KiCAD_Lib:BNO055; symbol BNO055:BNO055 -> SCR_KiCAD_Lib:BNO055
Changed lines of the file:
@@
 $EndComp
 $Comp
-L BNO055:BNO055 A2
+L SCR_KiCAD_Lib:BNO055 A2
 U 1 1 5E1FDF1C
 P 4900 3400
 F 0 "A2" H 4550 2950 50  0000 C CNN
 F 1 "BNO055" H 5150 2950 50  0000 C CNN
-F 2 "BNO055:BNO055" H 4900 3400 50  0001 C CNN
+F 2 "SCR_KiCAD_Lib:BNO055" H 4900 3400 50  0001 C CNN
 F 3 "" H 4900 3400 50  0001 C CNN
 	1    4900 3400

Commit message: Add connections to schematic
Connections:
- net labels added: L_Enable, L_Encoder_A, L_Encoder_B, L_IN_1, L_IN_2, L_Motor_+, L_Motor_-, R_Enable, R_Encoder_A, R_Encoder_B, R_IN_1, R_IN_2, SCL, SDA
Changed lines of the file:
@@
 	0    1    1    0
 $EndComp
+Text Label 8150 4400 0    50   ~ 0
+SCL
+Text Label 4400 3200 2    50   ~ 0
+SCL
+Text Label 8150 4300 0    50   ~ 0
+SDA
+Text Label 4400 3300 2    50   ~ 0
+SDA
+Text Label 4650 4350 2    50   ~ 0
+L_Motor_+
+Text Label 4650 5200 2    50   ~ 0
+L_Motor_+
+Text Label 4650 4450 2    50   ~ 0
+L_Motor_-
+Text Label 4650 5300 2    50   ~ 0
+L_Motor_-
+Text Label 4650 4750 2    50   ~ 0
+L_Encoder_A
+Text Label 7150 3500 2    50   ~ 0
+L_Encoder_A
+Text Label 5950 4800 2    50   ~ 0
+R_Encoder_A
+Text Label 7150 3600 2    50   ~ 0
+R_Encoder_A
+Text Label 4650 4850 2    50   ~ 0
+L_Encoder_B
+Text Label 5950 4900 2    50   ~ 0
+R_Encoder_B
+Text Label 7150 4400 2    50   ~ 0
+R_Encoder_B
+Text Label 7150 4500 2    50   ~ 0
+L_Encoder_B
+Text Label 5950 4400 2    50   ~ 0
+L_Motor_+
+Text Label 5950 4500 2    50   ~ 0
+L_Motor_-
+Text Label 5950 5250 2    50   ~ 0
+L_Motor_-
+Text Label 5950 5150 2    50   ~ 0
+L_Motor_+
+Text Label 6000 2700 2    50   ~ 0
+L_Enable
+Text Label 6000 2800 2    50   ~ 0
+L_IN_1
+Text Label 6000 2900 2    50   ~ 0
+L_IN_2
+Text Label 6500 2700 0    50   ~ 0
+R_Enable
+Text Label 6500 2800 0    50   ~ 0
+R_IN_1
+Text Label 6500 2900 0    50   ~ 0
+R_IN_2
+Text Label 7150 3700 2    50   ~ 0
+L_IN_1
+Text Label 7150 3800 2    50   ~ 0
+L_IN_2
+Text Label 7150 3900 2    50   ~ 0
+L_Enable
+Text Label 7150 4000 2    50   ~ 0
+R_IN_1
+Text Label 7150 4100 2    50   ~ 0
+R_IN_2
+Text Label 7150 4200 2    50   ~ 0
+R_Enable
 $EndSCHEMATC

Commit message: Update schematic and layout pcb
Parts:
- removed J1: Conn_01x04, symbol Connector_Generic:Conn_01x04
- added J1: Conn_01x02, Connector_JST:JST_EH_B2B-EH-A_1x02_P2.50mm_Vertical, symbol Connector_Generic:Conn_01x02
- J2: footprint (none) -> Connector_PinHeader_2.54mm:PinHeader_2x05_P2.54mm_Vertical
- J3, J4: footprint (none) -> Connector_PinHeader_2.54mm:PinHeader_1x06_P2.54mm_Vertical
- J5, J6: footprint (none) -> Connector_JST:JST_EH_B2B-EH-A_1x02_P2.50mm_Vertical
Connections:
- net labels added: R_Motor_+, R_Motor_-
Other:
- moved on the sheet: J3, J4
Changed lines of the file:
@@
 L Connector_Generic:Conn_01x06 J3
 U 1 1 5E201931
-P 4850 4550
-F 0 "J3" H 4930 4542 50  0000 L CNN
-F 1 "Conn_01x06" H 4930 4451 50  0000 L CNN
-F 2 "" H 4850 4550 50  0001 C CNN
-F 3 "~" H 4850 4550 50  0001 C CNN
-	1    4850 4550
+P 4600 4550
+F 0 "J3" H 4680 4542 50  0000 L CNN
+F 1 "Conn_01x06" H 4680 4451 50  0000 L CNN
+F 2 "Connector_PinHeader_2.54mm:PinHeader_1x06_P2.54mm_Vertical" H 4600 4550 50  0001 C CNN
+F 3 "~" H 4600 4550 50  0001 C CNN
+	1    4600 4550
 	1    0    0    -1
 $EndComp
@@
 L Connector_Generic:Conn_01x06 J4
 U 1 1 5E202B38
-P 6150 4600
-F 0 "J4" H 6230 4592 50  0000 L CNN
-F 1 "Conn_01x06" H 6230 4501 50  0000 L CNN
-F 2 "" H 6150 4600 50  0001 C CNN
-F 3 "~" H 6150 4600 50  0001 C CNN
-	1    6150 4600
+P 6200 4550
+F 0 "J4" H 6280 4542 50  0000 L CNN
+F 1 "Conn_01x06" H 6280 4451 50  0000 L CNN
+F 2 "Connector_PinHeader_2.54mm:PinHeader_1x06_P2.54mm_Vertical" H 6200 4550 50  0001 C CNN
+F 3 "~" H 6200 4550 50  0001 C CNN
+	1    6200 4550
 	1    0    0    -1
 $EndComp
@@
 L power:GND #PWR0105
 U 1 1 5E2046A5
-P 4650 4550
-F 0 "#PWR0105" H 4650 4300 50  0001 C CNN
-F 1 "GND" V 4655 4422 50  0000 R CNN
-F 2 "" H 4650 4550 50  0001 C CNN
-F 3 "" H 4650 4550 50  0001 C CNN
-	1    4650 4550
+P 4400 4550
+F 0 "#PWR0105" H 4400 4300 50  0001 C CNN
+F 1 "GND" V 4405 4422 50  0000 R CNN
+F 2 "" H 4400 4550 50  0001 C CNN
+F 3 "" H 4400 4550 50  0001 C CNN
+	1    4400 4550
 	0    1    1    0
 $EndComp
@@
 L power:+5V #PWR0106
 U 1 1 5E204AE1
-P 4650 4650
-F 0 "#PWR0106" H 4650 4500 50  0001 C CNN
-F 1 "+5V" V 4665 4778 50  0000 L CNN
-F 2 "" H 4650 4650 50  0001 C CNN
-F 3 "" H 4650 4650 50  0001 C CNN
-	1    4650 4650
+P 4400 4650
+F 0 "#PWR0106" H 4400 4500 50  0001 C CNN
+F 1 "+5V" V 4415 4778 50  0000 L CNN
+F 2 "" H 4400 4650 50  0001 C CNN
+F 3 "" H 4400 4650 50  0001 C CNN
+	1    4400 4650
 	0    -1   -1   0
 $EndComp
@@
 L power:+5V #PWR0107
 U 1 1 5E205184
-P 5950 4700
-F 0 "#PWR0107" H 5950 4550 50  0001 C CNN
-F 1 "+5V" V 5965 4828 50  0000 L CNN
-F 2 "" H 5950 4700 50  0001 C CNN
-F 3 "" H 5950 4700 50  0001 C CNN
-	1    5950 4700
+P 6000 4650
+F 0 "#PWR0107" H 6000 4500 50  0001 C CNN
+F 1 "+5V" V 6015 4778 50  0000 L CNN
+F 2 "" H 6000 4650 50  0001 C CNN
+F 3 "" H 6000 4650 50  0001 C CNN
+	1    6000 4650
 	0    -1   -1   0
 $EndComp
@@
 L power:GND #PWR0108
 U 1 1 5E2055A4
-P 5950 4600
-F 0 "#PWR0108" H 5950 4350 50  0001 C CNN
-F 1 "GND" V 5955 4472 50  0000 R CNN
-F 2 "" H 5950 4600 50  0001 C CNN
-F 3 "" H 5950 4600 50  0001 C CNN
-	1    5950 4600
+P 6000 4550
+F 0 "#PWR0108" H 6000 4300 50  0001 C CNN
+F 1 "GND" V 6005 4422 50  0000 R CNN
+F 2 "" H 6000 4550 50  0001 C CNN
+F 3 "" H 6000 4550 50  0001 C CNN
+	1    6000 4550
 	0    1    1    0
 $EndComp
@@
 F 0 "J2" H 6250 3217 50  0000 C CNN
 F 1 "Conn_02x05_Odd_Even" H 6250 3126 50  0000 C CNN
-F 2 "" H 6200 2800 50  0001 C CNN
+F 2 "Connector_PinHeader_2.54mm:PinHeader_2x05_P2.54mm_Vertical" H 6200 2800 50  0001 C CNN
 F 3 "~" H 6200 2800 50  0001 C CNN
 	1    6200 2800
@@
 NoConn ~ 7150 4600
 $Comp
-L Connector_Generic:Conn_01x02 J5
-U 1 1 5E20DAB0
-P 4850 5200
-F 0 "J5" H 4930 5192 50  0000 L CNN
-F 1 "Conn_01x02" H 4930 5101 50  0000 L CNN
-F 2 "" H 4850 5200 50  0001 C CNN
-F 3 "~" H 4850 5200 50  0001 C CNN
-	1    4850 5200
-	1    0    0    -1
-$EndComp
-$Comp
-L Connector_Generic:Conn_01x02 J6
-U 1 1 5E20E76D
-P 6150 5150
-F 0 "J6" H 6230 5142 50  0000 L CNN
-F 1 "Conn_01x02" H 6230 5051 50  0000 L CNN
-F 2 "" H 6150 5150 50  0001 C CNN
-F 3 "~" H 6150 5150 50  0001 C CNN
-	1    6150 5150
-	1    0    0    -1
-$EndComp
-$Comp
-L Connector_Generic:Conn_01x04 J1
-U 1 1 5E20F40F
-P 6150 3700
-F 0 "J1" H 6230 3692 50  0000 L CNN
-F 1 "Conn_01x04" H 6230 3601 50  0000 L CNN
-F 2 "" H 6150 3700 50  0001 C CNN
-F 3 "~" H 6150 3700 50  0001 C CNN
-	1    6150 3700
-	1    0    0    -1
-$EndComp
-$Comp
 L power:+5V #PWR0113
 U 1 1 5E20FCDA
-P 5950 3700
-F 0 "#PWR0113" H 5950 3550 50  0001 C CNN
-F 1 "+5V" V 5965 3828 50  0000 L CNN
-F 2 "" H 5950 3700 50  0001 C CNN
-F 3 "" H 5950 3700 50  0001 C CNN
-	1    5950 3700
-	0    -1   -1   0
-$EndComp
-$Comp
-L power:+5V #PWR0114
-U 1 1 5E210211
-P 5950 3800
-F 0 "#PWR0114" H 5950 3650 50  0001 C CNN
-F 1 "+5V" V 5965 3928 50  0000 L CNN
-F 2 "" H 5950 3800 50  0001 C CNN
-F 3 "" H 5950 3800 50  0001 C CNN
-	1    5950 3800
+P 4350 2400
+F 0 "#PWR0113" H 4350 2250 50  0001 C CNN
+F 1 "+5V" V 4365 2528 50  0000 L CNN
+F 2 "" H 4350 2400 50  0001 C CNN
+F 3 "" H 4350 2400 50  0001 C CNN
+	1    4350 2400
 	0    -1   -1   0
 $EndComp
@@
 L power:GND #PWR0115
 U 1 1 5E2104D1
-P 5950 3600
-F 0 "#PWR0115" H 5950 3350 50  0001 C CNN
-F 1 "GND" V 5955 3472 50  0000 R CNN
-F 2 "" H 5950 3600 50  0001 C CNN
-F 3 "" H 5950 3600 50  0001 C CNN
-	1    5950 3600
-	0    1    1    0
-$EndComp
-$Comp
-L power:GND #PWR0116
-U 1 1 5E210903
-P 5950 3900
-F 0 "#PWR0116" H 5950 3650 50  0001 C CNN
-F 1 "GND" V 5955 3772 50  0000 R CNN
-F 2 "" H 5950 3900 50  0001 C CNN
-F 3 "" H 5950 3900 50  0001 C CNN
-	1    5950 3900
+P 4350 2300
+F 0 "#PWR0115" H 4350 2050 50  0001 C CNN
+F 1 "GND" V 4355 2172 50  0000 R CNN
+F 2 "" H 4350 2300 50  0001 C CNN
+F 3 "" H 4350 2300 50  0001 C CNN
+	1    4350 2300
 	0    1    1    0
 $EndComp
@@
 Text Label 4400 3300 2    50   ~ 0
 SDA
-Text Label 4650 4350 2    50   ~ 0
+Text Label 4400 4450 2    50   ~ 0
 L_Motor_+
-Text Label 4650 5200 2    50   ~ 0
+Text Label 4400 5100 2    50   ~ 0
 L_Motor_+
-Text Label 4650 4450 2    50   ~ 0
+Text Label 4400 4350 2    50   ~ 0
 L_Motor_-
-Text Label 4650 5300 2    50   ~ 0
+Text Label 4400 5000 2    50   ~ 0
 L_Motor_-
-Text Label 4650 4750 2    50   ~ 0
+Text Label 4400 4750 2    50   ~ 0
 L_Encoder_A
 Text Label 7150 3500 2    50   ~ 0
 L_Encoder_A
-Text Label 5950 4800 2    50   ~ 0
+Text Label 6000 4750 2    50   ~ 0
 R_Encoder_A
 Text Label 7150 3600 2    50   ~ 0
 R_Encoder_A
-Text Label 4650 4850 2    50   ~ 0
+Text Label 4400 4850 2    50   ~ 0
 L_Encoder_B
-Text Label 5950 4900 2    50   ~ 0
+Text Label 6000 4850 2    50   ~ 0
 R_Encoder_B
 Text Label 7150 4400 2    50   ~ 0
@@
 Text Label 7150 4500 2    50   ~ 0
 L_Encoder_B
-Text Label 5950 4400 2    50   ~ 0
-L_Motor_+
-Text Label 5950 4500 2    50   ~ 0
-L_Motor_-
-Text Label 5950 5250 2    50   ~ 0
-L_Motor_-
-Text Label 5950 5150 2    50   ~ 0
-L_Motor_+
+Text Label 6000 4450 2    50   ~ 0
+R_Motor_+
+Text Label 6000 4350 2    50   ~ 0
+R_Motor_-
+Text Label 6000 5000 2    50   ~ 0
+R_Motor_-
 Text Label 6000 2700 2    50   ~ 0
 L_Enable
@@
 Text Label 7150 4200 2    50   ~ 0
 R_Enable
+Text Label 6000 5100 2    50   ~ 0
+R_Motor_+
+$Comp
+L Connector_Generic:Conn_01x02 J1
+U 1 1 5E2A7DCA
+P 4550 2300
+F 0 "J1" H 4630 2292 50  0000 L CNN
+F 1 "Conn_01x02" H 4630 2201 50  0000 L CNN
+F 2 "Connector_JST:JST_EH_B2B-EH-A_1x02_P2.50mm_Vertical" H 4550 2300 50  0001 C CNN
+F 3 "~" H 4550 2300 50  0001 C CNN
+	1    4550 2300
+	1    0    0    -1
+$EndComp
+$Comp
+L Connector_Generic:Conn_01x02 J5
+U 1 1 5E2A82DE
+P 4600 5000
+F 0 "J5" H 4680 4992 50  0000 L CNN
+F 1 "Conn_01x02" H 4680 4901 50  0000 L CNN
+F 2 "Connector_JST:JST_EH_B2B-EH-A_1x02_P2.50mm_Vertical" H 4600 5000 50  0001 C CNN
+F 3 "~" H 4600 5000 50  0001 C CNN
+	1    4600 5000
+	1    0    0    -1
+$EndComp
+$Comp
+L Connector_Generic:Conn_01x02 J6
+U 1 1 5E2A89E5
+P 6200 5000
+F 0 "J6" H 6280 4992 50  0000 L CNN
+F 1 "Conn_01x02" H 6280 4901 50  0000 L CNN
+F 2 "Connector_JST:JST_EH_B2B-EH-A_1x02_P2.50mm_Vertical" H 6200 5000 50  0001 C CNN
+F 3 "~" H 6200 5000 50  0001 C CNN
+	1    6200 5000
+	1    0    0    -1
+$EndComp
 $EndSCHEMATC

Commit message: Update connectors and layout
Parts:
- removed J1, J5, J6: Conn_01x02, Connector_JST:JST_EH_B2B-EH-A_1x02_P2.50mm_Vertical, symbol Connector_Generic:Conn_01x02
- removed J2: Conn_02x05_Odd_Even, Connector_PinHeader_2.54mm:PinHeader_2x05_P2.54mm_Vertical, symbol Connector_Generic:Conn_02x05_Odd_Even
- removed J3, J4: Conn_01x06, Connector_PinHeader_2.54mm:PinHeader_1x06_P2.54mm_Vertical, symbol Connector_Generic:Conn_01x06
- added J1, J2: Conn_01x05, Connector_JST:JST_XH_B5B-XH-A_1x05_P2.50mm_Vertical, symbol Connector_Generic:Conn_01x05
- added J3, J4: Conn_01x04, Connector_JST:JST_XH_B4B-XH-A_1x04_P2.50mm_Vertical, symbol Connector_Generic:Conn_01x04
Connections:
- net labels added: M1_Enable, M1_Encoder_A, M1_Encoder_B, M1_IN_1, M1_IN_2, M2_Enable, M2_Encoder_A, M2_Encoder_B, M2_IN_1, M2_IN_2
- net labels removed: L_Enable, L_Encoder_A, L_Encoder_B, L_IN_1, L_IN_2, L_Motor_+, L_Motor_-, R_Enable, R_Encoder_A, R_Encoder_B, R_IN_1, R_IN_2, R_Motor_+, R_Motor_-
- wire segments 2 -> 4
Other:
- note added: "Note: Power and communication is provided over USB\nThe Raspberry Pi delivers adaquate current for this application"
- moved on the sheet: A1
